Commit message: Aggiunta dell'algoritmo di navigazione

File: src/wamv_gazebo/urdf/model.urdf.xacro (robot description, xacro)
@@ -1,4 +1,5 @@
 <?xml version='1.0' encoding='utf-8'?>
-<robot name="wamv">
+<robot name="wamv" xmlns:xacro="http://ros.org/wiki/xacro">
+  <xacro:property name="user_path" value="file:///home/luca002/proj_ws/src/wamv_gazebo/models/wamv/meshes"/>
   <!-- BASE FOOTPRINT -->
   <link name="base_footprint" />
@@ -13,5 +14,5 @@
       <origin xyz="0 0 0" rpy="0 0 0" />
       <geometry>
-        <mesh filename="file:///home/luca002/proj_ws/src/wamv_gazebo/models/wamv/meshes/WAM-V-Base.dae" />
+        <mesh filename="${user_path}/WAM-V-Base.dae" />
       </geometry>
     </visual>
@@ -75,5 +76,5 @@
       <origin xyz="0 0 0" rpy="0 0 0" />
       <geometry>
-        <mesh filename="file:///home/luca002/proj_ws/src/wamv_gazebo/models/wamv/meshes/engine.dae" />
+        <mesh filename="${user_path}/engine.dae" />
       </geometry>
     </visual>
@@ -110,5 +111,5 @@
       <origin xyz="0 0 0" rpy="0 0 0" />
       <geometry>
-        <mesh filename="file:///home/luca002/proj_ws/src/wamv_gazebo/models/wamv/meshes/propeller.dae" />
+        <mesh filename="${user_path}/propeller.dae" />
       </geometry>
     </visual>
@@ -141,5 +142,5 @@
       <origin xyz="0 0 0" rpy="0 0 0" />
       <geometry>
-        <mesh filename="file:///home/luca002/proj_ws/src/wamv_gazebo/models/wamv/meshes/engine.dae" />
+        <mesh filename="${user_path}/engine.dae" />
       </geometry>
     </visual>
@@ -176,5 +177,5 @@
       <origin xyz="0 0 0" rpy="0 0 0"/>
       <geometry>
-        <mesh filename="file:///home/luca002/proj_ws/src/wamv_gazebo/models/wamv/meshes/propeller.dae"/>
+        <mesh filename="${user_path}/propeller.dae"/>
       </geometry>
     </visual>
@@ -207,5 +208,5 @@
       <origin xyz="0 0 0" rpy="0 0 0" />
       <geometry>
-        <mesh filename="file:///home/luca002/proj_ws/src/wamv_gazebo/models/wamv/meshes/battery.dae"/>
+        <mesh filename="${user_path}/battery.dae"/>
       </geometry>
     </visual>
@@ -234,5 +235,5 @@
       <origin xyz="0 0 0" rpy="0 0 0"/>
       <geometry>
-        <mesh filename="file:///home/luca002/proj_ws/src/wamv_gazebo/models/wamv/meshes/battery.dae"/>
+        <mesh filename="${user_path}/battery.dae"/>
       </geometry>
     </visual>
@@ -262,5 +263,5 @@
       <origin xyz="0 0 0" rpy="0 0 0"/>
       <geometry>
-        <mesh filename="file:///home/luca002/proj_ws/src/wamv_gazebo/models/wamv/meshes/cpu_cases.dae"/>
+        <mesh filename="${user_path}/cpu_cases.dae"/>
       </geometry>
     </visual>
@@ -296,5 +297,5 @@
       <origin xyz="0 0 0" rpy="0 0 0"/>
       <geometry>
-        <mesh filename="file:///home/luca002/proj_ws/src/wamv_gazebo/models/wamv/meshes/legs.dae" />
+        <mesh filename="${user_path}/legs.dae" />
       </geometry>
       <material name="dark_gray_metal">
@@ -326,5 +327,5 @@
       <origin xyz="0 0 0" rpy="0 0 0"/>
       <geometry>
-        <mesh filename="file:///home/luca002/proj_ws/src/wamv_gazebo/models/wamv/meshes/ring.dae"/>
+        <mesh filename="${user_path}/ring.dae"/>
       </geometry>
       <material name="gray_metal">
@@ -357,5 +358,5 @@
       <origin xyz="0 0 0" rpy="0 0 0"/>
       <geometry>
-        <mesh filename="file:///home/luca002/proj_ws/src/wamv_gazebo/models/wamv/meshes/lidar_3d_v1.dae"/>
+        <mesh filename="${user_path}/lidar_3d_v1.dae"/>
       </geometry>
     </visual>
@@ -376,5 +377,5 @@
     <sensor name="gpu_lidar" type="gpu_lidar">
       <pose>0 0 0.036 0 0 0</pose>
-      <update_rate>35</update_rate>
+      <update_rate>15</update_rate>
       <topic>scan</topic>
       <always_on>1</always_on>
@@ -386,6 +387,6 @@
             <samples>640</samples>
             <resolution>1</resolution>
-            <min_angle>-1.396263</min_angle>
-            <max_angle>1.396263</max_angle>
+            <min_angle>-1.570796</min_angle>
+            <max_angle>1.570796</max_angle>
           </horizontal>
           <vertical>
@@ -398,12 +399,7 @@
         <range>
           <min>0.08</min>
-          <max>30.0</max>
+          <max>50.0</max>
           <resolution>0.05</resolution>
         </range>
-        <noise>
-          <type>gaussian</type>
-          <mean>0.0</mean>
-          <stddev>0.0001</stddev>
-        </noise>
       </ray>
     </sensor>
@@ -447,4 +443,76 @@
             <noise type="gaussian">
               <mean>0</mean>
+              <stddev>0.008</stddev>               <!-- rumore standard leggermente ridotto -->
+              <bias_mean>0.0005</bias_mean>        <!-- bias medio realistico -->
+              <bias_stddev>0.003</bias_stddev>    <!-- deviazione bias -->
+              <dynamic_bias_stddev>0.000015</dynamic_bias_stddev>
+              <dynamic_bias_correlation_time>300.0</dynamic_bias_correlation_time>
+              <precision>0.0003</precision>
+            </noise>
+          </x>
+          <y>
+            <noise type="gaussian">
+              <mean>0</mean>
+              <stddev>0.008</stddev>
+              <bias_mean>0.0005</bias_mean>
+              <bias_stddev>0.003</bias_stddev>
+              <dynamic_bias_stddev>0.000015</dynamic_bias_stddev>
+              <dynamic_bias_correlation_time>300.0</dynamic_bias_correlation_time>
+              <precision>0.0003</precision>
+            </noise>
+          </y>
+          <z>
+            <noise type="gaussian">
+              <mean>0</mean>
+              <stddev>0.008</stddev>
+              <bias_mean>0.0005</bias_mean>
+              <bias_stddev>0.003</bias_stddev>
+              <dynamic_bias_stddev>0.000015</dynamic_bias_stddev>
+              <dynamic_bias_correlation_time>300.0</dynamic_bias_correlation_time>
+              <precision>0.0003</precision>
+            </noise>
+          </z>
+        </angular_velocity>
+        <linear_acceleration>
+          <x>
+            <noise type="gaussian">
+              <mean>0</mean>
+              <stddev>0.02</stddev>                 <!-- rumore standard realistico -->
+              <bias_mean>0.04</bias_mean>          <!-- bias medio -->
+              <bias_stddev>0.006</bias_stddev>    <!-- deviazione bias -->
+              <dynamic_bias_stddev>0.0003</dynamic_bias_stddev>
+              <dynamic_bias_correlation_time>150.0</dynamic_bias_correlation_time>
+              <precision>0.006</precision>
+            </noise>
+          </x>
+          <y>
+            <noise type="gaussian">
+              <mean>0</mean>
+              <stddev>0.02</stddev>
+              <bias_mean>0.04</bias_mean>
+              <bias_stddev>0.006</bias_stddev>
+              <dynamic_bias_stddev>0.0003</dynamic_bias_stddev>
+              <dynamic_bias_correlation_time>150.0</dynamic_bias_correlation_time>
+              <precision>0.006</precision>
+            </noise>
+          </y>
+          <z>
+            <noise type="gaussian">
+              <mean>0</mean>
+              <stddev>0.02</stddev>
+              <bias_mean>0.04</bias_mean>
+              <bias_stddev>0.006</bias_stddev>
+              <dynamic_bias_stddev>0.0003</dynamic_bias_stddev>
+              <dynamic_bias_correlation_time>150.0</dynamic_bias_correlation_time>
+              <precision>0.006</precision>
+            </noise>
+          </z>
+        </linear_acceleration>
+      </imu>
+      <!-- <imu>
+        <angular_velocity>
+          <x>
+            <noise type="gaussian">
+              <mean>0</mean>
               <stddev>0.009</stddev>
               <bias_mean>0.00075</bias_mean>
@@ -513,5 +581,5 @@
           </z>
         </linear_acceleration>
-      </imu>
+      </imu> -->
     </sensor>
   </gazebo>
@@ -601,14 +669,11 @@
   </gazebo>
   <gazebo>
-    <plugin
-      filename="gz-sim-odometry-publisher-system"
-      name="gz::sim::systems::OdometryPublisher">
+    <plugin filename="gz-sim-odometry-publisher-system" name="gz::sim::systems::OdometryPublisher">
       <odom_topic>/odom</odom_topic>
       <odom_frame>odom</odom_frame>
       <robot_base_frame>base_footprint</robot_base_frame>
       <dimension>2</dimension>
-      <publish_tf>false</publish_tf>
       <odom_publish_frequency>20.0</odom_publish_frequency>
-  </plugin>
+    </plugin>
   </gazebo>
 </robot>

Commit message: Aggiunta di commenti e modifiche

File: src/wamv_gazebo/urdf/model.urdf.xacro (robot description, xacro)
@@ -1,5 +1,5 @@
 <?xml version='1.0' encoding='utf-8'?>
 <robot name="wamv" xmlns:xacro="http://ros.org/wiki/xacro">
-  <xacro:property name="user_path" value="file:///home/luca002/proj_ws/src/wamv_gazebo/models/wamv/meshes"/>
+  <xacro:property name="user_path" value="file:///home/luca002/proj_ws/src/wamv_gazebo/urdf/meshes"/>
   <!-- BASE FOOTPRINT -->
   <link name="base_footprint" />
@@ -14,5 +14,5 @@
       <origin xyz="0 0 0" rpy="0 0 0" />
       <geometry>
-        <mesh filename="${user_path}/WAM-V-Base.dae" />
+        <mesh filename="${user_path}/wamv/WAM-V-Base.dae" />
       </geometry>
     </visual>
@@ -65,5 +65,5 @@
     <origin xyz="0 0 0" rpy="0 0 0" />
   </joint>
-  <!-- LEFT PART -->
+  <!-- WAM-V LEFT PART -->
   <!-- ENGINE -->
   <link name="left_engine_link">
@@ -76,5 +76,5 @@
       <origin xyz="0 0 0" rpy="0 0 0" />
       <geometry>
-        <mesh filename="${user_path}/engine.dae" />
+        <mesh filename="${user_path}/wamv/engine.dae" />
       </geometry>
     </visual>
@@ -111,5 +111,5 @@
       <origin xyz="0 0 0" rpy="0 0 0" />
       <geometry>
-        <mesh filename="${user_path}/propeller.dae" />
+        <mesh filename="${user_path}/wamv/propeller.dae" />
       </geometry>
     </visual>
@@ -129,5 +129,5 @@
     <origin xyz="-0.278156 0 -0.509371" rpy="0 0 0" />
   </joint>
-  <!-- RIGHT PART -->
+  <!-- WAM-V RIGHT PART -->
   <!-- ENGINE -->
   <link name="right_engine_link">
@@ -142,5 +142,5 @@
       <origin xyz="0 0 0" rpy="0 0 0" />
       <geometry>
-        <mesh filename="${user_path}/engine.dae" />
+        <mesh filename="${user_path}/wamv/engine.dae" />
       </geometry>
     </visual>
@@ -165,5 +165,5 @@
     <origin xyz="-2.373776 -1.027135 0.318237" rpy="0 0 0" />
   </joint>
-  <!-- PROPELLER -->0.15
+  <!-- PROPELLER -->
   <link name="right_propeller_link">
     <inertial>
@@ -177,5 +177,5 @@
       <origin xyz="0 0 0" rpy="0 0 0"/>
       <geometry>
-        <mesh filename="${user_path}/propeller.dae"/>
+        <mesh filename="${user_path}/wamv/propeller.dae"/>
       </geometry>
     </visual>
@@ -195,4 +195,5 @@
     <origin xyz="-0.278156 0 -0.509371" rpy="0 0 0" />
   </joint>
+  <!-- WAM-V LOAD -->
   <!-- BATTERIES -->
   <link name="battery_dx_link">
@@ -208,5 +209,5 @@
       <origin xyz="0 0 0" rpy="0 0 0" />
       <geometry>
-        <mesh filename="${user_path}/battery.dae"/>
+        <mesh filename="${user_path}/battery/battery.dae"/>
       </geometry>
     </visual>
@@ -235,5 +236,5 @@
       <origin xyz="0 0 0" rpy="0 0 0"/>
       <geometry>
-        <mesh filename="${user_path}/battery.dae"/>
+        <mesh filename="${user_path}/battery/battery.dae"/>
       </geometry>
     </visual>
@@ -263,5 +264,5 @@
       <origin xyz="0 0 0" rpy="0 0 0"/>
       <geometry>
-        <mesh filename="${user_path}/cpu_cases.dae"/>
+        <mesh filename="${user_path}/cpu_cases/cpu_cases.dae"/>
       </geometry>
     </visual>
@@ -297,5 +298,5 @@
       <origin xyz="0 0 0" rpy="0 0 0"/>
       <geometry>
-        <mesh filename="${user_path}/legs.dae" />
+        <mesh filename="${user_path}/tripod/legs.dae" />
       </geometry>
       <material name="dark_gray_metal">
@@ -327,5 +328,5 @@
       <origin xyz="0 0 0" rpy="0 0 0"/>
       <geometry>
-        <mesh filename="${user_path}/ring.dae"/>
+        <mesh filename="${user_path}/tripod/ring.dae"/>
       </geometry>
       <material name="gray_metal">
@@ -345,5 +346,4 @@
     <origin xyz="0 0 0.218" rpy="0 0 0" />
   </joint>
-  <!-- SENSORS -->
   <link name="lidar_link">
     <inertial>
@@ -358,5 +358,5 @@
       <origin xyz="0 0 0" rpy="0 0 0"/>
       <geometry>
-        <mesh filename="${user_path}/lidar_3d_v1.dae"/>
+        <mesh filename="${user_path}/lidar/lidar_3d_v1.dae"/>
       </geometry>
     </visual>
@@ -373,4 +373,5 @@
     <origin xyz="0 0 0.01" rpy="0 0 0" />
   </joint>
+  <!-- SENSORS -->
   <!-- LIDAR -->
   <gazebo reference="lidar_link">
@@ -443,7 +444,7 @@
             <noise type="gaussian">
               <mean>0</mean>
-              <stddev>0.008</stddev>               <!-- rumore standard leggermente ridotto -->
-              <bias_mean>0.0005</bias_mean>        <!-- bias medio realistico -->
-              <bias_stddev>0.003</bias_stddev>    <!-- deviazione bias -->
+              <stddev>0.008</stddev>
+              <bias_mean>0.0005</bias_mean>
+              <bias_stddev>0.003</bias_stddev>
               <dynamic_bias_stddev>0.000015</dynamic_bias_stddev>
               <dynamic_bias_correlation_time>300.0</dynamic_bias_correlation_time>
@@ -478,7 +479,7 @@
             <noise type="gaussian">
               <mean>0</mean>
-              <stddev>0.02</stddev>                 <!-- rumore standard realistico -->
-              <bias_mean>0.04</bias_mean>          <!-- bias medio -->
-              <bias_stddev>0.006</bias_stddev>    <!-- deviazione bias -->
+              <stddev>0.02</stddev>
+              <bias_mean>0.04</bias_mean>
+              <bias_stddev>0.006</bias_stddev>
               <dynamic_bias_stddev>0.0003</dynamic_bias_stddev>
               <dynamic_bias_correlation_time>150.0</dynamic_bias_correlation_time>
@@ -510,78 +511,7 @@
         </linear_acceleration>
       </imu>
-      <!-- <imu>
-        <angular_velocity>
-          <x>
-            <noise type="gaussian">
-              <mean>0</mean>
-              <stddev>0.009</stddev>
-              <bias_mean>0.00075</bias_mean>
-              <bias_stddev>0.005</bias_stddev>
-              <dynamic_bias_stddev>0.00002</dynamic_bias_stddev>
-              <dynamic_bias_correlation_time>400.0</dynamic_bias_correlation_time>
-              <precision>0.00025</precision>
-            </noise>
-          </x>
-          <y>
-            <noise type="gaussian">
-              <mean>0</mean>
-              <stddev>0.009</stddev>
-              <bias_mean>0.00075</bias_mean>
-              <bias_stddev>0.005</bias_stddev>
-              <dynamic_bias_stddev>0.00002</dynamic_bias_stddev>
-              <dynamic_bias_correlation_time>400.0</dynamic_bias_correlation_time>
-              <precision>0.00025</precision>
-            </noise>
-          </y>
-          <z>
-            <noise type="gaussian">
-              <mean>0</mean>
-              <stddev>0.009</stddev>
-              <bias_mean>0.00075</bias_mean>
-              <bias_stddev>0.005</bias_stddev>
-              <dynamic_bias_stddev>0.00002</dynamic_bias_stddev>
-              <dynamic_bias_correlation_time>400.0</dynamic_bias_correlation_time>
-              <precision>0.00025</precision>
-            </noise>
-          </z>
-        </angular_velocity>
-        <linear_acceleration>
-          <x>
-            <noise type="gaussian">
-              <mean>0</mean>
-              <stddev>0.021</stddev>
-              <bias_mean>0.05</bias_mean>
-              <bias_stddev>0.0075</bias_stddev>
-              <dynamic_bias_stddev>0.000375</dynamic_bias_stddev>
-              <dynamic_bias_correlation_time>175.0</dynamic_bias_correlation_time>
-              <precision>0.005</precision>
-            </noise>
-          </x>
-          <y>
-            <noise type="gaussian">
-              <mean>0</mean>
-              <stddev>0.021</stddev>
-              <bias_mean>0.05</bias_mean>
-              <bias_stddev>0.0075</bias_stddev>
-              <dynamic_bias_stddev>0.000375</dynamic_bias_stddev>
-              <dynamic_bias_correlation_time>175.0</dynamic_bias_correlation_time>
-              <precision>0.005</precision>
-            </noise>
-          </y>
-          <z>
-            <noise type="gaussian">
-              <mean>0</mean>
-              <stddev>0.021</stddev>
-              <bias_mean>0.05</bias_mean>
-              <bias_stddev>0.0075</bias_stddev>
-              <dynamic_bias_stddev>0.000375</dynamic_bias_stddev>
-              <dynamic_bias_correlation_time>175.0</dynamic_bias_correlation_time>
-              <precision>0.005</precision>
-            </noise>
-          </z>
-        </linear_acceleration>
-      </imu> -->
     </sensor>
   </gazebo>
+  <!-- PLUGINS -->
   <gazebo>
     <plugin name="gz::sim::systems::Thruster" filename="gz-sim-thruster-system">

Commit message: Adjustments

File: src/wamv_gazebo/urdf/model.urdf.xacro (robot description, xacro)
@@ -349,5 +349,5 @@
     <inertial>
       <origin xyz="0 0 0.036" rpy="0 0 0"/>
-      <mass value="0.83"/>
+      <mass value="1.2"/>
       <inertia
         ixx="0.001" ixy="0.0" ixz="0.0"
