Commit message: Eliche

File: install/wamv_gazebo/share/wamv_gazebo/urdf/model.urdf.xacro (robot description, xacro)
@@ -1 +1 @@
-/home/luca002/proj_ws/src/wamv_gazebo/urdf/model.urdf.xacro
+/home/gelatocotonato/LabMec2025/src/wamv_gazebo/urdf/model.urdf.xacro

File: src/wamv_gazebo/urdf/model.urdf.xacro (robot description, xacro)
@@ -1,5 +1,5 @@
 <?xml version='1.0' encoding='utf-8'?>
 <robot name="wamv" xmlns:xacro="http://ros.org/wiki/xacro">
-  <xacro:property name="user_path" value="file:///home/luca002/proj_ws/src/wamv_gazebo/urdf/meshes"/>
+  <xacro:property name="user_path" value="file:///home/gelatocotonato/LabMec2025/src/wamv_gazebo/urdf/meshes"/>
   <!-- BASE FOOTPRINT -->
   <link name="base_footprint" />
